File: tp_vino.kicad_pcb (KiCad board)
At the start: 2 copper layers, 96 parts, among them J1 TB_1X2, J10 PotO.Out, J2 TB_1X2, J3 TB_1X2, J4 TB_1X2, J5 TB_1X2, J6 V.RegOut, J7 Temp.Out, J8 C.RegOut, J9 PotTOut, P1 CONN_02X02, P10 3.3_GND_5V, P11 CONN_01X06, P12 CONN_01X06, P2 USB_OTG, P3 CONN_01X03, P4 Pot2_Out, P5 C.reg.in, P6 V_regOut, P7 Temp_Out, P8 C_RegOut, P9 PotO_Out, Q1 BC849, Q2 BC849, Q3 BC849, Q4 BC849, Q5 BC849, SW1 TEC_1, SW2 TEC_1, SW3 TEC_1, SW4 TEC_1, U1 ST3232E, U2 LM2576HVS-5, U3 NCP1117ST33T3G, U4 LM317_SOT223, U5 LM317_SOT223, U6 LM35-LP, U7 SIM800L

Commit message: Change names schematic.
Routing:
- net Net-(P2-Pad6): track 0.00 -> 18.3 mm
- net GND: track 519.6 -> 537.0 mm
Other:
- rule trace_min: 0.4 -> 0.2
Changed lines of the file:
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@@
   (general
     (links 185)
-    (no_connects 4)
+    (no_connects 0)
     (area 99.8019 57.829 221.768081 143.891681)
     (thickness 1.6)
     (drawings 6)
-    (tracks 746)
+    (tracks 757)
     (zones 0)
     (modules 96)
@@
   )
   (setup
-    (last_trace_width 1)
+    (last_trace_width 0.4)
     (user_trace_width 0.4)
     (user_trace_width 1)
@@
     (zone_clearance 0.508)
     (zone_45_only no)
-    (trace_min 0.4)
+    (trace_min 0.2)
     (segment_width 0.2)
     (edge_width 0.15)
@@
   (segment (start 121.412 115.824) (end 121.412 114.554) (width 1) (layer F.Cu) (net 5))
   (segment (start 120.166 117.07) (end 121.412 115.824) (width 1) (layer F.Cu) (net 5))
+  (segment (start 187.0456 96.647) (end 187.9981 96.647) (width 1) (layer F.Cu) (net 6))
+  (segment (start 187.9981 96.647) (end 190.4111 99.06) (width 1) (layer F.Cu) (net 6))
+  (segment (start 200.834 99.06) (end 202.692 97.202) (width 1) (layer F.Cu) (net 6))
+  (segment (start 190.4111 99.06) (end 200.834 99.06) (width 1) (layer F.Cu) (net 6))
   (segment (start 172.212 62.738) (end 172.2882 62.738) (width 1) (layer B.Cu) (net 6))
   (segment (start 172.2882 62.738) (end 173.8884 64.3382) (width 0.4) (layer B.Cu) (net 6))
@@
   (segment (start 112.014 108.204) (end 108.712 111.506) (width 1) (layer F.Cu) (net 14))
   (segment (start 108.712 111.506) (end 108.712 111.84) (width 0.6) (layer F.Cu) (net 14))
-  (segment (start 108.712 104.902) (end 114.3508 104.902) (width 1) (layer F.Cu) (net 15) (status 400000))
-  (segment (start 116.3828 106.934) (end 121.412 106.934) (width 1) (layer F.Cu) (net 15) (status 800000))
+  (segment (start 108.712 104.902) (end 114.3508 104.902) (width 1) (layer F.Cu) (net 15))
+  (segment (start 116.3828 106.934) (end 121.412 106.934) (width 1) (layer F.Cu) (net 15))
   (segment (start 114.3508 104.902) (end 116.3828 106.934) (width 1) (layer F.Cu) (net 15))
   (segment (start 108.712 104.902) (end 109.982 104.902) (width 0.25) (layer F.Cu) (net 15))
-  (segment (start 121.412 105.664) (end 117.4369 105.664) (width 1) (layer F.Cu) (net 16) (status 400000))
-  (segment (start 111.6749 99.902) (end 108.712 99.902) (width 1) (layer F.Cu) (net 16) (status 800000))
+  (segment (start 121.412 105.664) (end 117.4369 105.664) (width 1) (layer F.Cu) (net 16))
+  (segment (start 111.6749 99.902) (end 108.712 99.902) (width 1) (layer F.Cu) (net 16))
   (segment (start 117.4369 105.664) (end 111.6749 99.902) (width 1) (layer F.Cu) (net 16))
   (segment (start 108.712 99.902) (end 109.648 99.902) (width 0.25) (layer F.Cu) (net 16))
@@
   (segment (start 111.08944 68.9229) (end 113.3856 68.9229) (width 0.4) (layer F.Cu) (net 51))
   (segment (start 114.8389 67.4696) (end 114.8389 65.31654) (width 0.4) (layer F.Cu) (net 51))
+  (segment (start 117.0389 62.61654) (end 110.0389 62.61654) (width 0.4) (layer B.Cu) (net 55))
+  (segment (start 110.0389 62.61654) (end 110.0074 62.64804) (width 0.4) (layer B.Cu) (net 55))
+  (segment (start 110.0074 62.64804) (end 110.0074 64.28504) (width 0.4) (layer B.Cu) (net 55))
+  (segment (start 110.0074 64.28504) (end 111.0389 65.31654) (width 0.4) (layer B.Cu) (net 55))
+  (segment (start 111.0389 65.31654) (end 116.0389 65.31654) (width 0.4) (layer B.Cu) (net 55))
+  (segment (start 116.0389 65.31654) (end 117.0389 64.31654) (width 0.4) (layer B.Cu) (net 55))
+  (segment (start 117.0389 64.31654) (end 117.0389 62.61654) (width 0.4) (layer B.Cu) (net 55))
   (segment (start 202.692 121.58726) (end 202.692 116.586) (width 1) (layer F.Cu) (net 56))
   (segment (start 202.692 116.586) (end 198.2978 116.586) (width 1) (layer F.Cu) (net 56))
