File: RS232_TTL.sch (KiCad schematic (older format))
At the start: 11 parts, among them J1 TB_1X2, J2 TB_1X2, J3 TB_1X2, J4 TB_1X2, P1 CONN_02X02, U1 ST3232E

Commit message: Modifico algunos componentes. Seteo algunos encapsulados. Ordeno los componentes en el PCB.
Parts:
- C1, C2, C3, C4, C5: footprint ~ -> Capacitors_SMD:C_0805
- J1, J2, J3, J4: footprint (none) -> Connect:bornier2
- P1: footprint (none) -> Pin_Headers:Pin_Header_Straight_2x02
- U1: footprint (none) -> SMD_Packages:SO-16-N
Changed lines of the file:
@@
 EESchema Schematic File Version 2
 LIBS:tp_vino-cache
+LIBS:74xgxx
+LIBS:74xx
+LIBS:Altera
+LIBS:ESD_Protection
+LIBS:Lattice
+LIBS:Oscillators
+LIBS:Power_Management
+LIBS:Worldsemi
+LIBS:Xicor
+LIBS:Zilog
+LIBS:ac-dc
+LIBS:actel
+LIBS:adc-dac
+LIBS:analog_devices
+LIBS:analog_switches
+LIBS:atmel
+LIBS:audio
+LIBS:brooktre
+LIBS:cmos4000
+LIBS:cmos_ieee
+LIBS:conn
+LIBS:contrib
+LIBS:cypress
+LIBS:dc-dc
+LIBS:device
+LIBS:digital-audio
+LIBS:diode
+LIBS:display
+LIBS:dsp
+LIBS:elec-unifil
+LIBS:ftdi
+LIBS:gennum
+LIBS:graphic
+LIBS:hc11
+LIBS:intel
+LIBS:interface
+LIBS:ir
+LIBS:linear
+LIBS:logo
+LIBS:maxim
+LIBS:memory
+LIBS:microchip
+LIBS:microchip_dspic33dsc
+LIBS:microchip_pic10mcu
+LIBS:microchip_pic12mcu
+LIBS:microchip_pic16mcu
+LIBS:microchip_pic18mcu
+LIBS:microchip_pic32mcu
+LIBS:microcontrollers
+LIBS:motor_drivers
+LIBS:motorola
+LIBS:msp430
+LIBS:nordicsemi
+LIBS:nxp_armmcu
+LIBS:onsemi
+LIBS:opto
+LIBS:philips
+LIBS:power
+LIBS:powerint
+LIBS:pspice
+LIBS:references
+LIBS:regul
+LIBS:relays
+LIBS:rfcom
+LIBS:sensors
+LIBS:silabs
+LIBS:siliconi
+LIBS:stm8
+LIBS:stm32
+LIBS:supertex
+LIBS:switches
+LIBS:texas
+LIBS:transf
+LIBS:transistors
+LIBS:ttl_ieee
+LIBS:valves
+LIBS:video
+LIBS:xilinx
 EELAYER 25 0
 EELAYER END
@@
 F 0 "C1" V 3850 3150 30  0000 C CNN
 F 1 "100nF" V 3900 3200 30  0000 C CNN
-F 2 "~" H 3850 3050 60  0000 C CNN
+F 2 "Capacitors_SMD:C_0805" H 3850 3050 60  0001 C CNN
 F 3 "~" H 3850 3050 60  0000 C CNN
 	1    3850 3050
@@
 F 0 "C2" V 3850 3650 30  0000 C CNN
 F 1 "100nF" V 3900 3700 30  0000 C CNN
-F 2 "~" H 3850 3550 60  0000 C CNN
+F 2 "Capacitors_SMD:C_0805" H 3850 3550 60  0001 C CNN
 F 3 "~" H 3850 3550 60  0000 C CNN
 	1    3850 3550
@@
 F 0 "C4" H 5800 3400 30  0000 C CNN
 F 1 "100nF" H 5800 3350 30  0000 C CNN
-F 2 "~" H 5800 3250 60  0000 C CNN
+F 2 "Capacitors_SMD:C_0805" H 5800 3250 60  0001 C CNN
 F 3 "~" H 5800 3250 60  0000 C CNN
 	1    5800 3250
@@
 F 0 "C5" H 5800 3900 30  0000 C CNN
 F 1 "100nF" H 5800 3850 30  0000 C CNN
-F 2 "~" H 5800 3750 60  0000 C CNN
+F 2 "Capacitors_SMD:C_0805" H 5800 3750 60  0001 C CNN
 F 3 "~" H 5800 3750 60  0000 C CNN
 	1    5800 3750
@@
 F 0 "C3" V 5800 2950 30  0000 C CNN
 F 1 "100nF" V 5850 3000 30  0000 C CNN
-F 2 "~" H 5800 2850 60  0000 C CNN
+F 2 "Capacitors_SMD:C_0805" H 5800 2850 60  0001 C CNN
 F 3 "~" H 5800 2850 60  0000 C CNN
 	1    5800 2850
@@
 F 0 "U1" H 4800 4400 70  0000 C CNN
 F 1 "ST3232E" H 4800 2700 70  0000 C CNN
-F 2 "" H 4800 3550 60  0000 C CNN
+F 2 "SMD_Packages:SO-16-N" H 4800 3550 60  0001 C CNN
 F 3 "" H 4800 3550 60  0000 C CNN
 	1    4800 3550
@@
 F 0 "J4" H 6450 4350 60  0000 C CNN
 F 1 "TB_1X2" H 6500 3750 60  0000 C CNN
-F 2 "" H 6400 4100 60  0000 C CNN
+F 2 "Connect:bornier2" H 6400 4100 60  0001 C CNN
 F 3 "" H 6400 4100 60  0000 C CNN
 	1    6450 4050
@@
 F 0 "P1" H 3300 3650 50  0000 C CNN
 F 1 "CONN_02X02" H 3300 3350 50  0000 C CNN
-F 2 "" H 3300 2300 50  0000 C CNN
+F 2 "Pin_Headers:Pin_Header_Straight_2x02" H 3300 2300 50  0001 C CNN
 F 3 "" H 3300 2300 50  0000 C CNN
 	1    3300 3500
@@
 F 0 "J1" H 3100 4650 60  0000 C CNN
 F 1 "TB_1X2" H 3150 4050 60  0000 C CNN
-F 2 "" H 3050 4400 60  0000 C CNN
+F 2 "Connect:bornier2" H 3050 4400 60  0001 C CNN
 F 3 "" H 3050 4400 60  0000 C CNN
 	1    3100 4350
@@
 F 0 "J2" H 3800 5400 60  0000 C CNN
 F 1 "TB_1X2" H 3850 4800 60  0000 C CNN
-F 2 "" H 3750 5150 60  0000 C CNN
+F 2 "Connect:bornier2" H 3750 5150 60  0001 C CNN
 F 3 "" H 3750 5150 60  0000 C CNN
 	1    3800 5100
@@
 F 0 "J3" H 5750 5400 60  0000 C CNN
 F 1 "TB_1X2" H 5800 4800 60  0000 C CNN
-F 2 "" H 5700 5150 60  0000 C CNN
+F 2 "Connect:bornier2" H 5700 5150 60  0001 C CNN
 F 3 "" H 5700 5150 60  0000 C CNN
 	1    5750 5100

Commit message: Modificaciones en el schematic dado los componentes comprados empiezo a ordenar los componentes en una dimension estimada de 10x6 cm.
Parts:
- C1, C2, C3, C4, C5: footprint Capacitors_SMD:C_0805 -> Capacitors_SMD:C_1206
- J1, J2, J3, J4: footprint Connect:bornier2 -> Connect:AK300-2
Changed lines of the file:
@@
 F 0 "C1" V 3850 3150 30  0000 C CNN
 F 1 "100nF" V 3900 3200 30  0000 C CNN
-F 2 "Capacitors_SMD:C_0805" H 3850 3050 60  0001 C CNN
+F 2 "Capacitors_SMD:C_1206" H 3850 3050 60  0001 C CNN
 F 3 "~" H 3850 3050 60  0000 C CNN
 	1    3850 3050
@@
 F 0 "C2" V 3850 3650 30  0000 C CNN
 F 1 "100nF" V 3900 3700 30  0000 C CNN
-F 2 "Capacitors_SMD:C_0805" H 3850 3550 60  0001 C CNN
+F 2 "Capacitors_SMD:C_1206" H 3850 3550 60  0001 C CNN
 F 3 "~" H 3850 3550 60  0000 C CNN
 	1    3850 3550
@@
 F 0 "C4" H 5800 3400 30  0000 C CNN
 F 1 "100nF" H 5800 3350 30  0000 C CNN
-F 2 "Capacitors_SMD:C_0805" H 5800 3250 60  0001 C CNN
+F 2 "Capacitors_SMD:C_1206" H 5800 3250 60  0001 C CNN
 F 3 "~" H 5800 3250 60  0000 C CNN
 	1    5800 3250
@@
 F 0 "C5" H 5800 3900 30  0000 C CNN
 F 1 "100nF" H 5800 3850 30  0000 C CNN
-F 2 "Capacitors_SMD:C_0805" H 5800 3750 60  0001 C CNN
+F 2 "Capacitors_SMD:C_1206" H 5800 3750 60  0001 C CNN
 F 3 "~" H 5800 3750 60  0000 C CNN
 	1    5800 3750
@@
 $EndComp
 $Comp
-L GND-RESCUE-ciaa-nxp #PWR06
+L GND-RESCUE-ciaa-nxp #PWR08
 U 1 1 581A0FB6
 P 5950 3350
-F 0 "#PWR06" H 5950 3350 30  0001 C CNN
+F 0 "#PWR08" H 5950 3350 30  0001 C CNN
 F 1 "GND" H 5950 3280 30  0001 C CNN
 F 2 "" H 5950 3350 60  0000 C CNN
@@
 $EndComp
 $Comp
-L GND-RESCUE-ciaa-nxp #PWR07
+L GND-RESCUE-ciaa-nxp #PWR09
 U 1 1 581A0FB7
 P 5950 3850
-F 0 "#PWR07" H 5950 3850 30  0001 C CNN
+F 0 "#PWR09" H 5950 3850 30  0001 C CNN
 F 1 "GND" H 5950 3780 30  0001 C CNN
 F 2 "" H 5950 3850 60  0000 C CNN
@@
 F 0 "C3" V 5800 2950 30  0000 C CNN
 F 1 "100nF" V 5850 3000 30  0000 C CNN
-F 2 "Capacitors_SMD:C_0805" H 5800 2850 60  0001 C CNN
+F 2 "Capacitors_SMD:C_1206" H 5800 2850 60  0001 C CNN
 F 3 "~" H 5800 2850 60  0000 C CNN
 	1    5800 2850
@@
 $EndComp
 $Comp
-L GND-RESCUE-ciaa-nxp #PWR08
+L GND-RESCUE-ciaa-nxp #PWR010
 U 1 1 581A0FBA
 P 5650 3500
-F 0 "#PWR08" H 5650 3500 30  0001 C CNN
+F 0 "#PWR010" H 5650 3500 30  0001 C CNN
 F 1 "GND" H 5650 3430 30  0001 C CNN
 F 2 "" H 5650 3500 60  0000 C CNN
@@
 $EndComp
 $Comp
-L GND-RESCUE-ciaa-nxp #PWR09
+L GND-RESCUE-ciaa-nxp #PWR011
 U 1 1 581A0FBB
 P 5950 2950
-F 0 "#PWR09" H 5950 2950 30  0001 C CNN
+F 0 "#PWR011" H 5950 2950 30  0001 C CNN
 F 1 "GND" H 5950 2880 30  0001 C CNN
 F 2 "" H 5950 2950 60  0000 C CNN
@@
 $EndComp
 $Comp
-L +3.3V-RESCUE-ciaa-nxp #PWR010
+L +3.3V-RESCUE-ciaa-nxp #PWR012
 U 1 1 581A0FBC
 P 5650 2800
-F 0 "#PWR010" H 5650 2760 30  0001 C CNN
+F 0 "#PWR012" H 5650 2760 30  0001 C CNN
 F 1 "+3.3V" H 5650 2910 30  0000 C CNN
 F 2 "" H 5650 2800 60  0000 C CNN
@@
 F 0 "J4" H 6450 4350 60  0000 C CNN
 F 1 "TB_1X2" H 6500 3750 60  0000 C CNN
-F 2 "Connect:bornier2" H 6400 4100 60  0001 C CNN
+F 2 "Connect:AK300-2" H 6400 4100 60  0001 C CNN
 F 3 "" H 6400 4100 60  0000 C CNN
 	1    6450 4050
@@
 F 0 "J1" H 3100 4650 60  0000 C CNN
 F 1 "TB_1X2" H 3150 4050 60  0000 C CNN
-F 2 "Connect:bornier2" H 3050 4400 60  0001 C CNN
+F 2 "Connect:AK300-2" H 3050 4400 60  0001 C CNN
 F 3 "" H 3050 4400 60  0000 C CNN
 	1    3100 4350
@@
 F 0 "J2" H 3800 5400 60  0000 C CNN
 F 1 "TB_1X2" H 3850 4800 60  0000 C CNN
-F 2 "Connect:bornier2" H 3750 5150 60  0001 C CNN
+F 2 "Connect:AK300-2" H 3750 5150 60  0001 C CNN
 F 3 "" H 3750 5150 60  0000 C CNN
 	1    3800 5100
@@
 F 0 "J3" H 5750 5400 60  0000 C CNN
 F 1 "TB_1X2" H 5800 4800 60  0000 C CNN
-F 2 "Connect:bornier2" H 5700 5150 60  0001 C CNN
+F 2 "Connect:AK300-2" H 5700 5150 60  0001 C CNN
 F 3 "" H 5700 5150 60  0000 C CNN
 	1    5750 5100

Commit message: Modificaciones en el schematico.Cambio dimension a 10x7 cm.
Connections:
- net TTL_RS232_RXD1: now also P1.1 (P1); no longer P1.3 (P3)
- net TTL_RS232_TXD1: now also P1.3 (P3); no longer P1.1 (P1)
- net at J1.1, P1.2 (P2): now also U1.12 (R1OUT); no longer U1.11 (T1IN)
- net at J1.2, P1.4 (P4): now also U1.11 (T1IN); no longer U1.12 (R1OUT)
- net at U1.13 (R1IN): now also J4.2; no longer J4.1
- net at U1.14 (T1OUT): now also J4.1; no longer J4.2
Changed lines of the file:
@@
 Text Notes 7050 5150 0    60   ~ 0
 RS232
-Text HLabel 3250 3150 1    30   Input ~ 0
+Text HLabel 3350 3150 1    30   Input ~ 0
 TTL_RS232_RXD1
-Text HLabel 3350 3150 1    30   Output ~ 0
+Text HLabel 3250 3150 1    30   Output ~ 0
 TTL_RS232_TXD1
 $Comp
@@
 	1    5650 2800
 	1    0    0    -1
+$EndComp
+$Comp
+L TB_1X2 J4
+U 1 1 581A0FBD
+P 6450 4050
+F 0 "J4" H 6450 4350 60  0000 C CNN
+F 1 "TB_1X2" H 6500 3750 60  0000 C CNN
+F 2 "Connect:AK300-2" H 6400 4100 60  0001 C CNN
+F 3 "" H 6400 4100 60  0000 C CNN
+	1    6450 4050
+	-1   0    0    -1
+$EndComp
+$Comp
+L CONN_02X02 P1
+U 1 1 581A0FBE
+P 3300 3500
+F 0 "P1" H 3300 3650 50  0000 C CNN
+F 1 "CONN_02X02" H 3300 3350 50  0000 C CNN
+F 2 "Pin_Headers:Pin_Header_Straight_2x02" H 3300 2300 50  0001 C CNN
+F 3 "" H 3300 2300 50  0000 C CNN
+	1    3300 3500
+	0    1    1    0
+$EndComp
+$Comp
+L TB_1X2 J1
+U 1 1 581A0FBF
+P 3100 4350
+F 0 "J1" H 3100 4650 60  0000 C CNN
+F 1 "TB_1X2" H 3150 4050 60  0000 C CNN
+F 2 "Connect:AK300-2" H 3050 4400 60  0001 C CNN
+F 3 "" H 3050 4400 60  0000 C CNN
+	1    3100 4350
+	1    0    0    -1
+$EndComp
+$Comp
+L TB_1X2 J2
+U 1 1 581A0FC0
+P 3800 5100
+F 0 "J2" H 3800 5400 60  0000 C CNN
+F 1 "TB_1X2" H 3850 4800 60  0000 C CNN
+F 2 "Connect:AK300-2" H 3750 5150 60  0001 C CNN
+F 3 "" H 3750 5150 60  0000 C CNN
+	1    3800 5100
+	0    -1   -1   0
+$EndComp
+$Comp
+L TB_1X2 J3
+U 1 1 581A0FC1
+P 5750 5100
+F 0 "J3" H 5750 5400 60  0000 C CNN
+F 1 "TB_1X2" H 5800 4800 60  0000 C CNN
+F 2 "Connect:AK300-2" H 5700 5150 60  0001 C CNN
+F 3 "" H 5700 5150 60  0000 C CNN
+	1    5750 5100
+	0    -1   -1   0
 $EndComp
 Wire Wire Line
@@
 Wire Notes Line
 	2800 2200 2800 5300
-$Comp
-L TB_1X2 J4
-U 1 1 581A0FBD
-P 6450 4050
-F 0 "J4" H 6450 4350 60  0000 C CNN
-F 1 "TB_1X2" H 6500 3750 60  0000 C CNN
-F 2 "Connect:AK300-2" H 6400 4100 60  0001 C CNN
-F 3 "" H 6400 4100 60  0000 C CNN
-	1    6450 4050
-	-1   0    0    1
-$EndComp
 Wire Wire Line
 	5600 4050 5850 4050
-$Comp
-L CONN_02X02 P1
-U 1 1 581A0FBE
-P 3300 3500
-F 0 "P1" H 3300 3650 50  0000 C CNN
-F 1 "CONN_02X02" H 3300 3350 50  0000 C CNN
-F 2 "Pin_Headers:Pin_Header_Straight_2x02" H 3300 2300 50  0001 C CNN
-F 3 "" H 3300 2300 50  0000 C CNN
-	1    3300 3500
-	0    1    1    0
-$EndComp
-$Comp
-L TB_1X2 J1
-U 1 1 581A0FBF
-P 3100 4350
-F 0 "J1" H 3100 4650 60  0000 C CNN
-F 1 "TB_1X2" H 3150 4050 60  0000 C CNN
-F 2 "Connect:AK300-2" H 3050 4400 60  0001 C CNN
-F 3 "" H 3050 4400 60  0000 C CNN
-	1    3100 4350
-	1    0    0    -1
-$EndComp
-$Comp
-L TB_1X2 J2
-U 1 1 581A0FC0
-P 3800 5100
-F 0 "J2" H 3800 5400 60  0000 C CNN
-F 1 "TB_1X2" H 3850 4800 60  0000 C CNN
-F 2 "Connect:AK300-2" H 3750 5150 60  0001 C CNN
-F 3 "" H 3750 5150 60  0000 C CNN
-	1    3800 5100
-	0    -1   -1   0
-$EndComp
 Wire Wire Line
-	4000 3950 3350 3950
+	3550 4150 4000 4150
 Wire Wire Line
-	3350 3950 3350 3750
-Wire Wire Line
-	4000 4150 3600 4150
-Wire Wire Line
-	3600 4050 3600 4450
-Wire Wire Line
-	3600 4050 3250 4050
-Wire Wire Line
-	3250 4050 3250 3750
-Wire Wire Line
-	3450 4250 3500 4250
-Wire Wire Line
-	3500 4250 3500 3950
+	3500 3950 3500 4450
 Connection ~ 3500 3950
-Wire Wire Line
-	3600 4450 3450 4450
 Connection ~ 3600 4150
 Wire Wire Line
@@
 Wire Wire Line
 	3350 3150 3350 3250
-$Comp
-L TB_1X2 J3
-U 1 1 581A0FC1
-P 5750 5100
-F 0 "J3" H 5750 5400 60  0000 C CNN
-F 1 "TB_1X2" H 5800 4800 60  0000 C CNN
-F 2 "Connect:AK300-2" H 5700 5150 60  0001 C CNN
-F 3 "" H 5700 5150 60  0000 C CNN
-	1    5750 5100
-	0    -1   -1   0
-$EndComp
 Wire Wire Line
 	5650 4250 5650 4750
@@
 	5850 4050 5850 4750
 Wire Wire Line
-	5600 4150 6100 4150
+	3700 4050 4000 4050
+Wire Wire Line
+	5600 4250 5650 4250
+Wire Wire Line
+	3350 3750 3600 3750
+Wire Wire Line
+	3250 3950 4000 3950
+Wire Wire Line
+	3250 3950 3250 3750
+Wire Wire Line
+	3500 4450 3450 4450
+Wire Wire Line
+	3450 4250 3550 4250
+Wire Wire Line
+	3550 4250 3550 4150
+Wire Wire Line
+	3600 3750 3600 4150
 Wire Wire Line
 	6100 3950 5600 3950
 Wire Wire Line
-	3700 4050 4000 4050
-Wire Wire Line
-	5600 4250 5650 4250
+	5600 4150 6100 4150
 $EndSCHEMATC

Commit message: Change names schematic.
Parts:
- J1: value TB_1X2 -> TxRx_TTL1
- J2: value TB_1X2 -> TxRx_TTL2
- J3: value TB_1X2 -> TxRx232Out2
- J4: value TB_1X2 -> TxRx232Out1
- P1: value CONN_02X02 -> JmpSim
Changed lines of the file:
@@
 P 6450 4050
 F 0 "J4" H 6450 4350 60  0000 C CNN
-F 1 "TB_1X2" H 6500 3750 60  0000 C CNN
+F 1 "TxRx232Out1" H 6500 3750 60  0000 C CNN
 F 2 "Connect:AK300-2" H 6400 4100 60  0001 C CNN
 F 3 "" H 6400 4100 60  0000 C CNN
@@
 P 3300 3500
 F 0 "P1" H 3300 3650 50  0000 C CNN
-F 1 "CONN_02X02" H 3300 3350 50  0000 C CNN
+F 1 "JmpSim" H 3300 3350 50  0000 C CNN
 F 2 "Pin_Headers:Pin_Header_Straight_2x02" H 3300 2300 50  0001 C CNN
 F 3 "" H 3300 2300 50  0000 C CNN
@@
 P 3100 4350
 F 0 "J1" H 3100 4650 60  0000 C CNN
-F 1 "TB_1X2" H 3150 4050 60  0000 C CNN
+F 1 "TxRx_TTL1" H 3150 4050 60  0000 C CNN
 F 2 "Connect:AK300-2" H 3050 4400 60  0001 C CNN
 F 3 "" H 3050 4400 60  0000 C CNN
@@
 P 3800 5100
 F 0 "J2" H 3800 5400 60  0000 C CNN
-F 1 "TB_1X2" H 3850 4800 60  0000 C CNN
+F 1 "TxRx_TTL2" H 3850 4800 60  0000 C CNN
 F 2 "Connect:AK300-2" H 3750 5150 60  0001 C CNN
 F 3 "" H 3750 5150 60  0000 C CNN
@@
 P 5750 5100
 F 0 "J3" H 5750 5400 60  0000 C CNN
-F 1 "TB_1X2" H 5800 4800 60  0000 C CNN
+F 1 "TxRx232Out2" H 5800 4800 60  0000 C CNN
 F 2 "Connect:AK300-2" H 5700 5150 60  0001 C CNN
 F 3 "" H 5700 5150 60  0000 C CNN
