File: _autosave-tp_vino.kicad_pcb (KiCad board)
At the start: 2 copper layers, 101 x 70 mm, 96 parts, among them J1 TxRx_TTL1, J10 PotO.Out, J2 TxRx_TTL2, J3 TxRx232Out2, J4 TxRx232Out1, J5 Vin, J6 V.RegOut, J7 Temp.Out, J8 C.RegOut, J9 PotTOut, P1 JmpSim, P10 3.3v_GNF_5v, P11 SwPins, P12 PinLeds, P2 USB_OTG, P3 UartSim, P4 Pot2_Out, P5 C.reg.in, P6 V_regOut, P7 Temp_Out, P8 C_RegOut, P9 PotO_Out, Q1 BC849, Q2 BC849, Q3 BC849, Q4 BC849, Q5 BC849, SW1 TEC_1, SW2 TEC_1, SW3 TEC_1, SW4 TEC_1, U1 ST3232E, U2 LM2576HVS-5, U3 NCP1117ST33T3G, U4 LM317_SOT223, U5 LM317_SOT223, U6 LM35-LP, U7 SIM800L

Commit message: Add digikey code and comment schematic.
Changed lines of the file:
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@@
     (pad 6 thru_hole oval (at 3.4991 1.13746 270) (size 1.55 1) (drill oval 1.15 0.5) (layers *.Cu *.Mask F.SilkS)
       (net 55 "Net-(P2-Pad6)"))
-    (model ../../../../../home/lchico/Documents/Especializacion/Kicad_course/chz_hw_tp_vino/footprint/walter/conn_pc/usb_B_micro_smd.wrl
+    (model ${KIPRJMOD}/3d_files/usb_B_micro_smd.wrl
       (at (xyz 0 0 0))
       (scale (xyz 1 1 1))
@@
     (pad 1 thru_hole circle (at 0 0) (size 2.49936 2.49936) (drill 1.19888) (layers *.Cu *.Mask F.SilkS)
       (net 56 "Net-(RV3-Pad1)"))
-    (model Potentiometers.3dshapes/Potentiometer_Alps-RK163-single_15mm.wrl
+    (model ${KIPRJMOD}/3d_files/Potentiometer_Alps-RK163-single_15mm.wrl
       (at (xyz 0 -0.4 0))
       (scale (xyz 1 1 1))
@@
     (pad 15 smd rect (at -3.175 -3.175 90) (size 0.508 1.143) (layers F.Cu F.Paste F.Mask)
       (net 6 GND))
-    (model SMD_Packages.3dshapes/SO-16-N.wrl
+    (model ${KIPRJMOD}/3d_files/SO-16-N.wrl
       (at (xyz 0 0 0))
       (scale (xyz 0.5 0.4 0.5))
@@
     (pad 1 thru_hole circle (at 0 0 180) (size 1.524 1.524) (drill 0.8) (layers *.Cu *.Mask F.SilkS)
       (net 10 +5V))
-    (model TO_SOT_Packages_THT.3dshapes/TO-92_Inline_Wide.wrl
+    (model ${KIPRJMOD}/3d_files/TO-92_Inline_Wide.wrl
       (at (xyz 0.1 0 0))
       (scale (xyz 1 1 1))
@@
     (pad 2 smd rect (at 2.70002 0 270) (size 3.50012 2.30124) (layers F.Cu F.Paste F.Mask)
       (net 10 +5V))
-    (model Diodes_SMD.3dshapes/SMB_Handsoldering.wrl
+    (model ${KIPRJMOD}/3d_files/SMB_Handsoldering.wrl
       (at (xyz 0 0 0))
       (scale (xyz 0.3937 0.3937 0.3937))
@@
     (pad 2 smd rect (at 2.05 0.8 270) (size 0.9 1) (layers F.Cu F.Paste F.Mask)
       (net 6 GND))
-    (model /home/lchico/Especialidad/Proyecto/Hardware/tp_vino/footprint/switch/switch/pcb_push2.wrl
+    (model ${KIPRJMOD}/3d_files/pcb_push2.wrl
       (at (xyz 0 0 0))
       (scale (xyz 1 1 1))
@@
     (pad 2 smd rect (at 2.05 0.8 270) (size 0.9 1) (layers F.Cu F.Paste F.Mask)
       (net 6 GND))
-    (model /home/lchico/Especialidad/Proyecto/Hardware/tp_vino/footprint/switch/switch/smd_push2.wrl
+    (model ${KIPRJMOD}/3d_files/smd_push2.wrl
       (at (xyz 0 0 0))
       (scale (xyz 1 1 1))
@@
     (pad 2 smd rect (at 2.05 0.8 270) (size 0.9 1) (layers F.Cu F.Paste F.Mask)
       (net 6 GND))
-    (model /home/lchico/Especialidad/Proyecto/Hardware/tp_vino/footprint/switch/switch/smd_push2.wrl
+    (model ${KIPRJMOD}/3d_files/smd_push2.wrl
       (at (xyz 0 0 0))
       (scale (xyz 1 1 1))
@@
     (pad 2 smd rect (at 2.05 0.8 270) (size 0.9 1) (layers F.Cu F.Paste F.Mask)
       (net 6 GND))
-    (model /home/lchico/Especialidad/Proyecto/Hardware/tp_vino/footprint/switch/switch/smd_push2.wrl
+    (model ${KIPRJMOD}/3d_files/smd_push2.wrl
       (at (xyz 0 0 0))
       (scale (xyz 1 1 1))
@@
     (pad 1 smd rect (at 0 -3.4 180) (size 4.6 1.1) (layers F.Cu F.Paste F.Mask)
       (net 9 "Net-(C6-Pad1)"))
-    (model TO_SOT_Packages_SMD.3dshapes/TO-263-5Lead.wrl
+    (model ${KIPRJMOD}/3d_files/TO-263-5Lead.wrl
       (at (xyz 0 0 0))
       (scale (xyz 1 1 1))
@@
     (pad 6 thru_hole oval (at 0 12.7 270) (size 2.032 1.7272) (drill 1.016) (layers *.Cu *.Mask F.SilkS)
       (net 6 GND))
-    (model Pin_Headers.3dshapes/Pin_Header_Straight_1x06.wrl
+    (model ${KIPRJMOD}/3d_files/Pin_Header_Straight_1x06.wrl
       (at (xyz 0 -0.25 0))
       (scale (xyz 1 1 1))
@@
     (pad 6 thru_hole oval (at 0 12.7 270) (size 2.032 1.7272) (drill 1.016) (layers *.Cu *.Mask F.SilkS)
       (net 6 GND))
-    (model Pin_Headers.3dshapes/Pin_Header_Straight_1x06.wrl
+    (model ${KIPRJMOD}/3d_files/Pin_Header_Straight_1x06.wrl
       (at (xyz 0 -0.25 0))
       (scale (xyz 1 1 1))
@@
     (pad 3 smd rect (at 0 -0.99822 270) (size 0.8001 0.8001) (layers F.Cu F.Paste F.Mask)
       (net 58 "Net-(Q2-Pad3)"))
-    (model TO_SOT_Packages_SMD.3dshapes/SOT-23.wrl
+    (model ${KIPRJMOD}/3d_files/SOT-23.wrl
       (at (xyz 0 0 0))
       (scale (xyz 1 1 1))
@@
     (pad 3 smd rect (at 0 -0.99822 180) (size 0.8001 0.8001) (layers F.Cu F.Paste F.Mask)
       (net 60 "Net-(Q3-Pad3)"))
-    (model TO_SOT_Packages_SMD.3dshapes/SOT-23.wrl
+    (model ${KIPRJMOD}/3d_files/SOT-23.wrl
       (at (xyz 0 0 0))
       (scale (xyz 1 1 1))
@@
     (pad 3 smd rect (at 0 -0.99822) (size 0.8001 0.8001) (layers F.Cu F.Paste F.Mask)
       (net 62 "Net-(Q4-Pad3)"))
-    (model TO_SOT_Packages_SMD.3dshapes/SOT-23.wrl
+    (model ${KIPRJMOD}/3d_files/SOT-23.wrl
       (at (xyz 0 0 0))
       (scale (xyz 1 1 1))
@@
     (pad 3 smd rect (at 0 -0.99822 90) (size 0.8001 0.8001) (layers F.Cu F.Paste F.Mask)
       (net 64 "Net-(Q5-Pad3)"))
-    (model TO_SOT_Packages_SMD.3dshapes/SOT-23.wrl
+    (model ${KIPRJMOD}/3d_files/SOT-23.wrl
       (at (xyz 0 0 0))
       (scale (xyz 1 1 1))
@@
     (pad 4 thru_hole oval (at 2.54 2.54) (size 1.7272 1.7272) (drill 1.016) (layers *.Cu *.Mask F.SilkS)
       (net 28 "Net-(P5-Pad2)"))
-    (model Pin_Headers.3dshapes/Pin_Header_Straight_2x02.wrl
+    (model ${KIPRJMOD}/3d_files/Pin_Header_Straight_2x02.wrl
       (at (xyz 0.05 -0.05 0))
       (scale (xyz 1 1 1))
@@
     (pad 2 thru_hole oval (at 0 2.54 90) (size 2.032 2.032) (drill 1.016) (layers *.Cu *.Mask F.SilkS)
       (net 6 GND))
-    (model Pin_Headers.3dshapes/Pin_Header_Straight_1x02.wrl
+    (model ${KIPRJMOD}/3d_files/Pin_Header_Straight_1x02.wrl
       (at (xyz 0 -0.05 0))
       (scale (xyz 1 1 1))
@@
     (pad 2 thru_hole oval (at 0 2.54 180) (size 2.032 2.032) (drill 1.016) (layers *.Cu *.Mask F.SilkS)
       (net 6 GND))
-    (model Pin_Headers.3dshapes/Pin_Header_Straight_1x02.wrl
+    (model ${KIPRJMOD}/3d_files/Pin_Header_Straight_1x02.wrl
       (at (xyz 0 -0.05 0))
       (scale (xyz 1 1 1))
@@
     (pad 3 thru_hole oval (at 0 5.08 270) (size 2.032 1.7272) (drill 1.016) (layers *.Cu *.Mask F.SilkS)
       (net 5 +3.3V))
-    (model Pin_Headers.3dshapes/Pin_Header_Straight_1x03.wrl
+    (model ${KIPRJMOD}/3d_files/Pin_Header_Straight_1x03.wrl
       (at (xyz 0 -0.1 0))
       (scale (xyz 1 1 1))
@@
     (pad 2 smd rect (at 1.651 0 90) (size 1.524 2.032) (layers F.Cu F.Paste F.Mask)
       (net 69 "Net-(R27-Pad2)"))
-    (model SMD_Packages.3dshapes/SMD-1206_Pol.wrl
+    (model ${KIPRJMOD}/3d_files/SMD-1206_Pol.wrl
       (at (xyz 0 0 0))
       (scale (xyz 0.17 0.16 0.16))
@@
     (pad 2 thru_hole oval (at 5 0 90) (size 1.9812 3.9624) (drill 1.3208) (layers *.Cu F.Paste F.SilkS F.Mask)
       (net 6 GND))
-    (model Terminal_Blocks.3dshapes/Pheonix_MKDS1.5-2pol.wrl
+    (model 3d_files/Pheonix_MKDS1.5-2pol.wrl
       (at (xyz 0.1 0 0))
       (scale (xyz 1 1 1))
@@
   (segment (start 126.6698 91.26982) (end 129.032 93.63202) (width 1) (layer F.Cu) (net 10))
   (segment (start 121.92 88.47) (end 125.427 88.47) (width 1) (layer F.Cu) (net 10))
-  (segment (start 131.5466 79.9846) (end 128.778 77.216) (width 0.4) (layer B.Cu) (net 10))
-  (segment (start 131.5466 91.11742) (end 131.5466 79.9846) (width 0.4) (layer B.Cu) (net 10))
-  (segment (start 129.032 93.63202) (end 131.5466 91.11742) (width 0.4) (layer B.Cu) (net 10))
+  (segment (start 131.5466 79.9846) (end 128.778 77.216) (width 1) (layer B.Cu) (net 10))
+  (segment (start 131.5466 91.11742) (end 131.5466 79.9846) (width 1) (layer B.Cu) (net 10))
+  (segment (start 129.032 93.63202) (end 131.5466 91.11742) (width 1) (layer B.Cu) (net 10))
   (segment (start 139.7 115.824) (end 139.7 114.0333) (width 1) (layer B.Cu) (net 10))
   (segment (start 144.8943 92.0496) (end 139.8524 87.0077) (width 1) (layer B.Cu) (net 10))
@@
   (segment (start 154.5844 78.4733) (end 154.5336 78.5241) (width 0.4) (layer F.Cu) (net 77))
   (via (at 154.5844 78.4733) (size 0.6) (drill 0.4) (layers F.Cu B.Cu) (net 77))
-  (segment (start 182.8546 78.4733) (end 154.5844 78.4733) (width 0.4) (layer B.Cu) (net 77))
-  (segment (start 186.9186 82.5373) (end 182.8546 78.4733) (width 0.4) (layer B.Cu) (net 77))
+  (segment (start 182.8546 78.4733) (end 154.5844 78.4733) (width 1) (layer B.Cu) (net 77))
+  (segment (start 186.9186 82.5373) (end 182.8546 78.4733) (width 1) (layer B.Cu) (net 77))
   (segment (start 186.9186 84.9376) (end 186.9186 82.5373) (width 1) (layer B.Cu) (net 77))
   (segment (start 188.5061 86.5251) (end 186.9186 84.9376) (width 1) (layer B.Cu) (net 77))
@@
     (connect_pads (clearance 0.508))
     (min_thickness 0.254)
-    (fill yes (arc_segments 16) (thermal_gap 0.508) (thermal_bridge_width 0.508))
+    (fill (arc_segments 16) (thermal_gap 0.508) (thermal_bridge_width 0.508))
     (polygon
       (pts
@@
     (connect_pads (clearance 0.508))
     (min_thickness 0.254)
-    (fill yes (arc_segments 16) (thermal_gap 0.508) (thermal_bridge_width 0.508))
+    (fill (arc_segments 16) (thermal_gap 0.508) (thermal_bridge_width 0.508))
     (polygon
       (pts
